Commit message: fix rviz error .05 value in sick model

File: elektron_description/urdf/sensors/sick_laser_lmx_100.urdf (robot description, URDF)
Before this commit: robot None, 1 links, 1 joints
Links:
- link base_laser_link: geometry collision cylinder length=0.05 radius=0.05; visual mesh filename=package://elektron_description/meshes/sensors/laser/sick_lm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
